File: _autosave-Samochodzik.kicad_pcb (KiCad board)
At the start: 2 copper layers, 63.5 x 92.5 mm, 101 parts, among them J1 MOT1, J10 GPIO_HD_3, J11 JUMP_GPIO5, J12 GPIO_HD_4, J13 JUMP_GPIO12, J14 VBAT, J15 JUMP_GPIO5, J16 EXP_IO1, J17 JUMP_GPIO5, J18 JUMP_GPIO5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

Commit message: DRC errors corrected
Routing:
- net GND: vias 55 -> 73
